Commit message: inclusion of optical frame

File: urdf/darwin.urdf (robot description, URDF)
Before this commit: robot darwinOP, 31 links, 30 joints
Links:
- added link MP_CAM_OPTICAL_FRAME
Joints:
- added joint j_cam_optical_frame: type fixed, parent MP_HEAD, child MP_CAM_OPTICAL_FRAME, origin xyz=-0.050000 -0.010000 0.000000 rpy=0.000000 -1.5708 0.000000, axis 0 0 1

Commit message: Adding sole_r and sole_r frames

File: urdf/darwin.urdf (robot description, URDF)
Before this commit: robot darwinOP, 32 links, 31 joints
Links:
- added link MP_SOLE_L
- added link MP_SOLE_R
Joints:
- added joint j_sole_l: type fixed, parent MP_ANKLE2_L, child MP_SOLE_L, origin xyz=-0.033500 -0.000000 0.000000 rpy=0.000000 0.000000 0.000000, axis 0 0 1
- added joint j_sole_r: type fixed, parent MP_ANKLE2_R, child MP_SOLE_R, origin xyz=0.033500 -0.000000 0.000000 rpy=0.000000 0.000000 0.000000, axis 0 0 1

Commit message: correction of r_sole and l_sole's coordinate system

File: urdf/darwin.urdf (robot description, URDF)
Before this commit: robot darwinOP, 34 links, 33 joints
Joints:
- joint j_sole_l: origin xyz=-0.033500 -0.000000 0.000000 rpy=0.000000 0.000000 0.000000 -> xyz=-0.033500 -0.000000 0.000000 rpy=0.000000 -1.5708 3.1416
- joint j_sole_r: origin xyz=0.033500 -0.000000 0.000000 rpy=0.000000 0.000000 0.000000 -> xyz=0.033500 -0.000000 0.000000 rpy=0.000000 -1.5708 0.000000
